Commit message: Fix incorrect joint coordinates for left and right eyes

File: oreo/assembly/assembly.urdf (robot description, URDF)
Before this commit: robot oreo_assembly, 5 links, 4 joints
Links:
- added link left_eye_link, mass 99.78e-3; visual mesh filename=file:///home/oreo/Documents/oreo_sim/oreo/assembly/stl/left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
- added link left_eye_yolk_link, mass 26.61e-3; visual mesh filename=file:///home/oreo/Documents/oreo_sim/oreo/assembly/stl/left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
- added link right_eye_link, mass 99.77e-3; visual mesh filename=file:///home/oreo/Documents/oreo_sim/oreo/assembly/stl/righ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
- added link right_eye_yolk_link, mass 26.61e-3; visual mesh filename=file:///home/oreo/Documents/oreo_sim/oreo/assembly/stl/righ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
- link base_link: geometry visual mesh filename=file:///home/oreo/Documents/oreo_sim/oreo/assembly/stl/Base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
- link neck_link: geometry visual mesh filename=file:///home/oreo/Documents/oreo_sim/oreo/assembly/stl/Neck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
- link pitch_piece_link: geometry visual mesh filename=file:///home/oreo/Documents/oreo_sim/oreo/assembly/stl/pitc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
- link skull_link: geometry visual mesh filename=file:///home/oreo/Documents/oreo_sim/oreo/assembly/stl/Skul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
Joints:
- added joint left_eye_joint: type continuous, parent left_eye_yolk_link, child left_eye_link, origin xyz=0 18.45e-3 45.97e-3 rpy=0 0 0, axis 0 0 1
- added joint left_eye_yolk_joint: type continuous, parent skull_link, child left_eye_yolk_link, origin xyz=52e-3 29e-3 -24.96e-3 rpy=0 0 0, axis 0 0 1
- added joint right_eye_link: type continuous, parent right_eye_yolk_link, child right_eye_link, origin xyz=0 -18.45e-3 45.97e-3 rpy=0 0 0, axis 0 0 1
- added joint right_eye_yolk_joint: type continuous, parent skull_link, child right_eye_yolk_link, origin xyz=52e-3 -29e-3 -24.96e-3 rpy=0 0 0, axis 0 0 1
