Commit message: Initial working copy simulating oreo robot in pybullet (omits roll movement of head, and missing some constraints in the eye/yolk asm)

File: oreo/sim/assembly.urdf (robot description, URDF)
Before this commit: robot oreo_assembly, 17 links, 16 joints
Links:
- link base_link: geometry collision mesh filename=stl/Base_asm.STL; visual mesh filename=stl/Base_asm.STL
- link dogbone_link_far_left: geometry collision mesh filename=stl/dogbone.STL; visual mesh filename=stl/dogbone.STL
- link dogbone_link_far_right: geometry collision mesh filename=stl/dogbone.STL; visual mesh filename=stl/dogbone.STL
- link dogbone_link_mid_left: geometry collision mesh filename=stl/dogbone.STL; visual mesh filename=stl/dogbone.STL
- link dogbone_link_mid_right: geometry collision mesh filename=stl/dogbone.STL; visual mesh filename=stl/dogbone.STL
- link left_eye_link: geometry collision mesh filename=stl/left_eye_asm.STL; visual mesh filename=stl/left_eye_asm.STL
- link left_eye_yolk_link: geometry collision mesh filename=stl/left_eye_yolk_asm.STL; visual mesh filename=stl/left_eye_yolk_asm.STL
- link linear_motor_rod_link_far_left: geometry collision mesh filename=stl/linear_motor_rod_assembly.STL; visual mesh filename=stl/linear_motor_rod_assembly.STL
- link linear_motor_rod_link_far_right: geometry collision mesh filename=stl/linear_motor_rod_assembly.STL; visual mesh filename=stl/linear_motor_rod_assembly.STL
- link linear_motor_rod_link_mid_left: geometry collision mesh filename=stl/linear_motor_rod_assembly.STL; visual mesh filename=stl/linear_motor_rod_assembly.STL
- link linear_motor_rod_link_mid_right: geometry collision mesh filename=stl/linear_motor_rod_assembly.STL; visual mesh filename=stl/linear_motor_rod_assembly.STL
- link neck_link: geometry collision mesh filename=stl/Neck_asm.STL; visual mesh filename=stl/Neck_asm.STL
- link pitch_piece_link: geometry collision mesh filename=stl/pitch_piece.STL; visual mesh filename=stl/pitch_piece.STL
- link right_eye_link: geometry collision mesh filename=stl/right_eye_asm.STL; visual mesh filename=stl/right_eye_asm.STL
- link right_eye_yolk_link: geometry collision mesh filename=stl/right_eye_yolk_asm.STL; visual mesh filename=stl/right_eye_yolk_asm.STL
- link skull_link: geometry collision mesh filename=stl/Skull.STL; visual mesh filename=stl/Skull.STL
Joints:
- joint base_joint: origin (none) -> xyz=0 0 0 rpy=0 0 0
- joint dogbone_joint_far_left: axis 0 0 1 -> (none); origin xyz=79.09e-3 0 0 rpy=3.1415 -0.566 -0.06 -> xyz=79.77e-3 0 0 rpy=3.1415 -0.566 0
- joint dogbone_joint_far_right: axis 0 0 1 -> (none); origin xyz=79.09e-3 0 0 rpy=0 0.566 0.06 -> xyz=79.77e-3 0 0 rpy=0 0.566 0
- joint dogbone_joint_mid_left: axis 0 0 1 -> (none); origin xyz=79.09e-3 0 0 rpy=3.1415 -0.566 -0.06 -> xyz=79.77e-3 0 0 rpy=3.1415 -0.566 0
- joint dogbone_joint_mid_right: axis 0 0 1 -> (none); origin xyz=79.09e-3 0 0 rpy=0 0.566 0.06 -> xyz=79.77e-3 0 0 rpy=0 0.566 0
- joint left_eye_joint: axis 0 0 1 -> 0 1 0
- joint right_eye_joint: axis 0 0 1 -> 0 1 0
- joint skull_joint: axis 1 0 0 -> (none); type continuous -> fixed

File: oreo/sim/assembly_temp.urdf (robot description, URDF)
Before this commit: robot oreo_assembly, 17 links, 16 joints
Joints:
- joint dogbone_joint_far_left: axis 0 0 1 -> (none); type continuous -> spherical
- joint dogbone_joint_far_right: axis 0 0 1 -> (none); type continuous -> spherical
- joint dogbone_joint_mid_left: axis 0 0 1 -> (none); type continuous -> spherical
- joint dogbone_joint_mid_right: axis 0 0 1 -> (none); type continuous -> spherical

Commit message: Added roll movement of skull assembly

File: oreo/sim/assembly.urdf (robot description, URDF)
Before this commit: robot oreo_assembly, 17 links, 16 joints
Joints:
- joint skull_joint: axis (none) -> 1 0 0; type fixed -> continuous

Commit message: added mpc work, cleaned up repo

File: oreo/sim/assembly.urdf (robot description, URDF)
Before this commit: robot oreo_assembly, 17 links, 16 joints
Joints:
- joint linear_motor_rod_joint_far_right: type prismatic -> fixed
- joint linear_motor_rod_joint_mid_right: type prismatic -> fixed
- joint neck_joint: type continuous -> fixed
- joint pitch_piece_joint: type continuous -> fixed
- joint skull_joint: type continuous -> fixed
